File: 7BitCounter.sch (KiCad schematic (older format))
At the start: 1 part, among them U2 NTE4024

Commit message: Update
Connections:
- net Q6: now reaches U2.3 (Q6)
- net Q5: now reaches U2.4 (Q5)
- net Q4: now reaches U2.5 (Q4)
- net Qf renamed Q3
Changed lines of the file:
@@
 $Descr A4 11693 8268
 encoding utf-8
-Sheet 3 3
+Sheet 3 4
 Title ""
 Date ""
@@
 	7650 2550 7850 2550
 Text HLabel 7850 2650 2    50   Output ~ 0
-Qf
+Q3
 Wire Wire Line
 	7650 2650 7850 2650
+Text HLabel 7850 2750 2    50   Output ~ 0
+Q4
+Text HLabel 7850 2850 2    50   Output ~ 0
+Q5
+Text HLabel 7850 2950 2    50   Output ~ 0
+Q6
+Wire Wire Line
+	7650 2750 7850 2750
+Wire Wire Line
+	7650 2850 7850 2850
+Wire Wire Line
+	7650 2950 7850 2950
 $EndSCHEMATC

Commit message: Added: pcb
Parts:
- U2: footprint (none) -> Package_DIP:DIP-14_W7.62mm
Changed lines of the file:
@@
 F 0 "U2" H 7250 3350 50  0000 C CNN
 F 1 "NTE4024" H 7250 3250 50  0000 C CNN
-F 2 "" H 7100 2700 50  0001 C CNN
+F 2 "Package_DIP:DIP-14_W7.62mm" H 7100 2700 50  0001 C CNN
 F 3 "" H 7100 2700 50  0001 C CNN
 	1    7100 2700
