File: ClockProvider.sch (KiCad schematic (older format))
At the start: 5 parts, among them U1 LM555

Commit message: Added: pcb
Parts:
- C1: footprint (none) -> Capacitor_THT:CP_Radial_D4.0mm_P1.50mm
- C2: footprint (none) -> Capacitor_THT:C_Disc_D3.0mm_W1.6mm_P2.50mm
- R1, R2: footprint (none) -> Resistor_THT:R_Axial_DIN0204_L3.6mm_D1.6mm_P1.90mm_Vertical
- U1: footprint (none) -> Package_DIP:DIP-8_W7.62mm
Changed lines of the file:
@@
 F 0 "U1" H 5250 3081 50  0000 C CNN
 F 1 "LM555" H 5250 2990 50  0000 C CNN
-F 2 "" H 5250 2500 50  0001 C CNN
+F 2 "Package_DIP:DIP-8_W7.62mm" H 5250 2500 50  0001 C CNN
 F 3 "http://www.ti.com/lit/ds/symlink/lm555.pdf" H 5250 2500 50  0001 C CNN
 	1    5250 2500
@@
 F 0 "R2" H 6520 2596 50  0000 L CNN
 F 1 "5k" H 6520 2505 50  0000 L CNN
-F 2 "" V 6380 2550 50  0001 C CNN
+F 2 "Resistor_THT:R_Axial_DIN0204_L3.6mm_D1.6mm_P1.90mm_Vertical" V 6380 2550 50  0001 C CNN
 F 3 "~" H 6450 2550 50  0001 C CNN
 	1    6450 2550
@@
 F 0 "R1" H 6520 2296 50  0000 L CNN
 F 1 "10k" H 6520 2205 50  0000 L CNN
-F 2 "" V 6380 2250 50  0001 C CNN
+F 2 "Resistor_THT:R_Axial_DIN0204_L3.6mm_D1.6mm_P1.90mm_Vertical" V 6380 2250 50  0001 C CNN
 F 3 "~" H 6450 2250 50  0001 C CNN
 	1    6450 2250
@@
 F 0 "C1" H 6628 2996 50  0000 L CNN
 F 1 "47uF" H 6628 2905 50  0000 L CNN
-F 2 "" H 6450 2950 50  0001 C CNN
+F 2 "Capacitor_THT:CP_Radial_D4.0mm_P1.50mm" H 6450 2950 50  0001 C CNN
 F 3 "~" H 6450 2950 50  0001 C CNN
 	1    6450 2950
@@
 F 0 "C2" H 3950 2800 50  0000 L CNN
 F 1 "10nf" H 3950 2700 50  0000 L CNN
-F 2 "" H 4300 2750 50  0001 C CNN
+F 2 "Capacitor_THT:C_Disc_D3.0mm_W1.6mm_P2.50mm" H 4300 2750 50  0001 C CNN
 F 3 "~" H 4300 2750 50  0001 C CNN
 	1    4300 2750
