File: ClockProvider.sch (KiCad schematic (older format))
At the start: 5 parts, among them U1 LM555

Commit message: Added: Mounting holes
Parts:
- C1: footprint Capacitor_THT:CP_Radial_D4.0mm_P1.50mm -> Capacitor_THT:C_Disc_D3.0mm_W1.6mm_P2.50mm
Changed lines of the file:
@@
 F 0 "C1" H 6628 2996 50  0000 L CNN
 F 1 "47uF" H 6628 2905 50  0000 L CNN
-F 2 "Capacitor_THT:CP_Radial_D4.0mm_P1.50mm" H 6450 2950 50  0001 C CNN
+F 2 "Capacitor_THT:C_Disc_D3.0mm_W1.6mm_P2.50mm" H 6450 2950 50  0001 C CNN
 F 3 "~" H 6450 2950 50  0001 C CNN
 	1    6450 2950
