File: LedDriver.sch (KiCad schematic (older format))
At the start: 6 parts

Commit message: Added: Mounting holes
Parts:
- R3, R4, R5: renamed from R?; footprint (none) -> Resistor_THT:R_Axial_DIN0204_L3.6mm_D1.6mm_P1.90mm_Vertical
- gave numbers to parts that had none: 3
Connections:
- net Aout: now reaches Q1.3 (C)
- net Bout: now reaches Q2.3 (C)
- net Cout: now reaches Q3.3 (C)
Changed lines of the file:
@@
 $Descr A4 11693 8268
 encoding utf-8
-Sheet 5 5
+Sheet 4 5
 Title ""
 Date ""
@@
 U 1 1 5D152BEF
 P 5550 1600
-F 0 "Q?" H 5741 1646 50  0000 L CNN
+AR Path="/5D152BEF" Ref="Q?"  Part="1"
+AR Path="/5D1523E9/5D152BEF" Ref="Q1"  Part="1"
+F 0 "Q1" H 5741 1646 50  0000 L CNN
 F 1 "PN2222A" H 5741 1555 50  0000 L CNN
 F 2 "Package_TO_SOT_THT:TO-92_Inline" H 5750 1525 50  0001 L CIN
@@
 P 5550 2150
 AR Path="/5D152BF5" Ref="Q?"  Part="1"
-AR Path="/5D1523E9/5D152BF5" Ref="Q?"  Part="1"
-F 0 "Q?" H 5741 2196 50  0000 L CNN
+AR Path="/5D1523E9/5D152BF5" Ref="Q2"  Part="1"
+F 0 "Q2" H 5741 2196 50  0000 L CNN
 F 1 "PN2222A" H 5741 2105 50  0000 L CNN
 F 2 "Package_TO_SOT_THT:TO-92_Inline" H 5750 2075 50  0001 L CIN
@@
 P 5550 2700
 AR Path="/5D152BFB" Ref="Q?"  Part="1"
-AR Path="/5D1523E9/5D152BFB" Ref="Q?"  Part="1"
-F 0 "Q?" H 5741 2746 50  0000 L CNN
+AR Path="/5D1523E9/5D152BFB" Ref="Q3"  Part="1"
+F 0 "Q3" H 5741 2746 50  0000 L CNN
 F 1 "PN2222A" H 5741 2655 50  0000 L CNN
 F 2 "Package_TO_SOT_THT:TO-92_Inline" H 5750 2625 50  0001 L CIN
@@
 	5800 2350 5800 1800
 $Comp
-L power:GND #PWR?
+L power:GND #PWR08
 U 1 1 5D15914C
 P 5650 3050
-F 0 "#PWR?" H 5650 2800 50  0001 C CNN
+F 0 "#PWR08" H 5650 2800 50  0001 C CNN
 F 1 "GND" H 5655 2877 50  0000 C CNN
 F 2 "" H 5650 3050 50  0001 C CNN
@@
 Wire Wire Line
 	5650 3050 5650 3100
-Text Notes 6300 1400 0    50   ~ 0
+Text Notes 5350 1150 0    50   ~ 0
 R=120/Ic\n
 $Comp
-L Device:R R?
+L Device:R R3
 U 1 1 5D159BAF
 P 5100 1600
-F 0 "R?" V 4893 1600 50  0000 C CNN
+F 0 "R3" V 4893 1600 50  0000 C CNN
 F 1 "R" V 4984 1600 50  0000 C CNN
-F 2 "" V 5030 1600 50  0001 C CNN
+F 2 "Resistor_THT:R_Axial_DIN0204_L3.6mm_D1.6mm_P1.90mm_Vertical" V 5030 1600 50  0001 C CNN
 F 3 "~" H 5100 1600 50  0001 C CNN
 	1    5100 1600
@@
 $EndComp
 $Comp
-L Device:R R?
+L Device:R R4
 U 1 1 5D15A660
 P 5100 2150
-F 0 "R?" V 4893 2150 50  0000 C CNN
+F 0 "R4" V 4893 2150 50  0000 C CNN
 F 1 "R" V 4984 2150 50  0000 C CNN
-F 2 "" V 5030 2150 50  0001 C CNN
+F 2 "Resistor_THT:R_Axial_DIN0204_L3.6mm_D1.6mm_P1.90mm_Vertical" V 5030 2150 50  0001 C CNN
 F 3 "~" H 5100 2150 50  0001 C CNN
 	1    5100 2150
@@
 $EndComp
 $Comp
-L Device:R R?
+L Device:R R5
 U 1 1 5D15A8D8
 P 5100 2700
-F 0 "R?" V 4893 2700 50  0000 C CNN
+F 0 "R5" V 4893 2700 50  0000 C CNN
 F 1 "R" V 4984 2700 50  0000 C CNN
-F 2 "" V 5030 2700 50  0001 C CNN
+F 2 "Resistor_THT:R_Axial_DIN0204_L3.6mm_D1.6mm_P1.90mm_Vertical" V 5030 2700 50  0001 C CNN
 F 3 "~" H 5100 2700 50  0001 C CNN
 	1    5100 2700
@@
 Wire Wire Line
 	4950 1600 4800 1600
+Text HLabel 6050 1400 2    50   Output ~ 0
+Aout
+Wire Wire Line
+	5650 1400 6050 1400
+Text HLabel 6050 1950 2    50   Output ~ 0
+Bout
+Wire Wire Line
+	5650 1950 6050 1950
+Text HLabel 6050 2500 2    50   Output ~ 0
+Cout
+Wire Wire Line
+	6050 2500 5650 2500
 $EndSCHEMATC
